Commit message: added inertial tags for simulation

File: franka_description/robots/panda_arm.xacro (robot description, xacro)
@@ -11,4 +11,7 @@
       </joint>
     </xacro:unless>
+    <!-- for simulation -->
+    <xacro:property name="joint_damping" value="0.0"/>
+    <!-- end for simulation -->
     <link name="${arm_id}_link0">
       <visual>
@@ -35,4 +38,11 @@
         </geometry>
       </collision>
+      <!-- for simulation -->
+      <inertial>
+        <origin xyz="0 0 0" rpy="0 0 0" />
+        <mass value="5.0" />
+        <inertia ixx="0.0" ixy="0.0" ixz="0.0" iyy="0.0" iyz="0.0" izz="0.0" />
+      </inertial>
+      <!-- end for simulation -->
     </link>
     <link name="${arm_id}_link1">
@@ -60,4 +70,11 @@
         </geometry>
       </collision>
+      <!-- for simulation -->
+      <inertial>
+        <origin xyz="0.0038 0.0021 -0.1750" rpy="0 0 0" />
+        <mass value="4.9707" />
+        <inertia ixx="0.7034" ixy="-0.0001" ixz="0.0068" iyy="0.7066" iyz="0.0197" izz="0.0091" />
+      </inertial>
+      <!-- end for simulation -->
     </link>
     <joint name="${arm_id}_joint1" type="revolute">
@@ -68,4 +85,7 @@
       <axis xyz="0 0 1"/>
       <limit effort="87" lower="-2.8973" upper="2.8973" velocity="2.1750"/>
+      <!-- for simulation -->
+      <dynamics damping="${joint_damping}" friction="0.546"/>
+      <!-- end for simulation -->
     </joint>
     <link name="${arm_id}_link2">
@@ -93,4 +113,10 @@
         </geometry>
       </collision>
+      <!-- for simulation -->
+      <inertial>
+        <origin xyz="-0.0031 -0.0287 0.0034" rpy="0 0 0" />
+        <mass value="0.6469" />
+        <inertia ixx="0.0080" ixy="-0.0039" ixz="0.0103" iyy="0.0281" iyz="0.0007" izz="0.0260" />
+      </inertial>
     </link>
     <joint name="${arm_id}_joint2" type="revolute">
@@ -101,4 +127,7 @@
       <axis xyz="0 0 1"/>
       <limit effort="87" lower="-1.7628" upper="1.7628" velocity="2.1750"/>
+      <!-- for simulation -->
+      <dynamics damping="${joint_damping}" friction="0.87224"/>
+      <!-- end for simulation -->
     </joint>
     <link name="${arm_id}_link3">
@@ -126,4 +155,11 @@
         </geometry>
       </collision>
+      <!-- for simulation -->
+      <inertial>
+        <origin xyz="0.0275 0.0392 -0.0665" rpy="0 0 0" />
+        <mass value="3.2286" />
+        <inertia ixx="0.0372" ixy="-0.0047" ixz="-0.0011" iyy="0.03615" iyz="-0.0128" izz="0.0108" />
+      </inertial>
+      <!-- end for simulation -->
     </link>
     <joint name="${arm_id}_joint3" type="revolute">
@@ -134,4 +170,7 @@
       <axis xyz="0 0 1"/>
       <limit effort="87" lower="-2.8973" upper="2.8973" velocity="2.1750"/>
+      <!-- for simulation -->
+      <dynamics damping="${joint_damping}" friction="0.6406"/>
+      <!-- end for simulation -->
     </joint>
     <link name="${arm_id}_link4">
@@ -159,4 +198,11 @@
         </geometry>
       </collision>
+      <!-- for simulation -->
+      <inertial>
+        <origin xyz="-0.0532 0.1044 0.0274" rpy="0 0 0" />
+        <mass value="3.5879" />
+        <inertia ixx="0.0259" ixy="0.0078" ixz="-0.0013" iyy="0.0195" iyz="0.0086" izz="0.0283" />
+      </inertial>
+      <!-- end for simulation -->
     </link>
     <joint name="${arm_id}_joint4" type="revolute">
@@ -167,4 +213,7 @@
       <axis xyz="0 0 1"/>
       <limit effort="87" lower="-3.0718" upper="-0.0698" velocity="2.1750"/>
+      <!-- for simulation -->
+      <dynamics damping="${joint_damping}" friction="1.2794"/>
+      <!-- end for simulation -->
     </joint>
     <link name="${arm_id}_link5">
@@ -210,4 +259,11 @@
         </geometry>
       </collision>
+      <!-- for simulation -->
+      <inertial>
+        <origin xyz="-0.0532 0.1044 0.0274" rpy="0 0 0" />
+        <mass value="1.2259" />
+        <inertia ixx="0.0355" ixy="-0.0021" ixz="-0.0040" iyy="0.0294" iyz="0.0002" izz="0.0086" />
+      </inertial>
+      <!-- end for simulation -->
     </link>
     <joint name="${arm_id}_joint5" type="revolute">
@@ -218,4 +274,7 @@
       <axis xyz="0 0 1"/>
       <limit effort="12" lower="-2.8973" upper="2.8973" velocity="2.6100"/>
+      <!-- for simulation -->
+      <dynamics damping="${joint_damping}" friction="0.839"/>
+      <!-- end for simulation -->
     </joint>
     <link name="${arm_id}_link6">
@@ -243,4 +302,11 @@
         </geometry>
       </collision>
+      <!-- for simulation -->
+      <inertial>
+        <origin xyz="0.0601 -0.0141 -0.0105" rpy="0 0 0" />
+        <mass value="1.6665" />
+        <inertia ixx="0.0196" ixy="0.0001" ixz="-0.0011" iyy="0.0043" iyz="0.0003" izz="0.0054" />
+      </inertial>
+      <!-- end for simulation -->
     </link>
     <joint name="${arm_id}_joint6" type="revolute">
@@ -251,4 +317,7 @@
       <axis xyz="0 0 1"/>
       <limit effort="12" lower="-0.0175" upper="3.7525" velocity="2.6100"/>
+      <!-- for simulation -->
+      <dynamics damping="${joint_damping}" friction="0.303"/>
+      <!-- end for simulation -->
     </joint>
     <link name="${arm_id}_link7">
@@ -276,4 +345,9 @@
         </geometry>
       </collision>
+      <inertial>
+        <origin xyz="0.0105 -0.0043 0.0616" rpy="0 0 0" />
+        <mass value="0.7355" />
+        <inertia ixx="0.0125" ixy="-0.0004" ixz="-0.0012" iyy="0.0100" iyz="-0.0007" izz="0.0048" />
+      </inertial>
     </link>
     <joint name="${arm_id}_joint7" type="revolute">
@@ -284,4 +358,7 @@
       <axis xyz="0 0 1"/>
       <limit effort="12" lower="-2.8973" upper="2.8973" velocity="2.6100"/>
+      <!-- for simulation -->
+      <dynamics damping="${joint_damping}" friction="0.5649"/>
+      <!-- end for simulation -->
     </joint>
     <link name="${arm_id}_link8">
@@ -304,4 +381,11 @@
         </geometry>
       </collision>
+      <!-- for simulation -->
+      <inertial>
+        <origin xyz="0 0 0" rpy="0 0 0" />
+        <mass value="0.1" />
+        <inertia ixx="0.0" ixy="0.0" ixz="0.0" iyy="0.0" iyz="0.0" izz="0.0" />
+      </inertial>
+      <!-- end for simulation -->
     </link>
     <joint name="${arm_id}_joint8" type="fixed">
